File: hardware/flight-computer/memory.kicad_sch (KiCad schematic)
At the start: 5 parts, among them U8 W25Q128JVS

Commit message: Worked on tidy up just pyro and sd card to go
Connections:
- net SCK renamed MCU_SCK
- net SDI renamed MCU_SDI
- net SDO renamed MCU_SDO
Changed lines of the file:
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@@
 		)
 	)
-	(hierarchical_label "SDI"
+	(hierarchical_label "MCU_SDI"
 		(shape output)
 		(at 106.68 106.68 180)
@@
 		)
 	)
-	(hierarchical_label "SDO"
+	(hierarchical_label "MCU_SDO"
 		(shape input)
 		(at 106.68 104.14 180)
@@
 		)
 	)
-	(hierarchical_label "SCK"
+	(hierarchical_label "MCU_SCK"
 		(shape input)
 		(at 106.68 101.6 180)
